Commit message: add shell tf. add sleep to save battery add default mac id

File: sphero_description/urdf/sphero.urdf (robot description, URDF)
Before this commit: robot sphero, 1 links, 0 joints
Links:
- added link shell, mass 0.5; collision sphere radius=0.0381; visual mesh filename=package://sphero_description/meshes/Sphero_Textured.dae scale=1.3 1.3 1.3
- link base_link: geometry collision sphere radius=0.0281; visual sphere radius=0.0381
Joints:
- added joint shell_joint: type floating, parent base_link, child shell, origin xyz=0 0 0 rpy=0 0 0
